File: controller/controller.kicad_pcb (KiCad board)
At the start: 2 copper layers, 18 parts, among them J1 USB_B, J2 Conn_01x03, SW1 Rotary_Encoder_Switch, SW2 Rotary_Encoder_Switch, SW3 Rotary_Encoder_Switch, U1 STM32F030F4Px, U2 RT9193, X2 SWD

Commit message: WIP
Parts:
- moved H4 124.7 mm to (99.0, 71.0)
- moved H2 86.2 mm to (99.0, 49.0)
- moved U1 69.9 mm to (156.0, 51.0)
- moved U2 62.6 mm to (124.0, 51.6), turned to 90 degrees
- moved C6 60.3 mm to (120.0, 51.0), turned to 270 degrees
- moved J1 54.8 mm to (126.0, 60.0), turned to 270 degrees
- moved X2 52.7 mm to (169.0, 47.0), turned to 180 degrees
- moved C1 51.2 mm to (150.0, 49.0), turned to 90 degrees
- moved C5 49.1 mm to (128.0, 51.0), turned to 270 degrees
- moved H1 48.4 mm to (181.0, 71.0)
- moved C4 47.1 mm to (124.0, 56.0), turned to 180 degrees
- moved H3 47.0 mm to (181.0, 49.0)
- moved J2 47.0 mm to (152.5, 65.0), turned to 0 degrees
- moved C2 46.8 mm to (162.0, 51.0), turned to 270 degrees
- moved C3 45.5 mm to (150.0, 53.0), turned to 90 degrees
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Routing:
- net Net-(SW1-PadS1): track 0.00 -> 67.8 mm, vias 0 -> 2
- net Net-(SW1-PadA): track 0.00 -> 65.1 mm, vias 0 -> 2
- net +3V3: track 0.00 -> 59.0 mm
- net +5V: track 0.00 -> 57.2 mm
- net Net-(SW1-PadB): track 0.00 -> 56.2 mm, vias 0 -> 2
- net GND: track 0.00 -> 25.5 mm, vias 0 -> 6
- net Net-(SW2-PadA): track 0.00 -> 24.9 mm
- net Net-(SW2-PadS1): track 0.00 -> 24.8 mm, vias 0 -> 2
- net Net-(SW3-PadB): track 0.00 -> 23.6 mm
- net /SWDIO: track 0.00 -> 20.0 mm, vias 0 -> 2
- net Net-(SW3-PadS1): track 0.00 -> 19.9 mm, vias 0 -> 1
- net Net-(SW3-PadA): track 0.00 -> 19.5 mm
- net Net-(SW2-PadB): track 0.00 -> 18.4 mm
- net /LED_DATA: track 0.00 -> 18.0 mm
- net /SWCLK: track 0.00 -> 12.7 mm, vias 0 -> 1
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- added copper zone on B.Cu, net GND
Other:
- board outline added: 90 x 30 mm
- net class Default: trace_width 0.25 -> 0.4
- board text added: "RINGLE v1.0 special design for KLADNÝ ZUBAŘ"
