File: controller/controller.kicad_pcb (KiCad board)
At the start: 2 copper layers, 90 x 30 mm, 18 parts, among them J1 USB_B, J2 Conn_01x03, SW1 Rotary_Encoder_Switch, SW2 Rotary_Encoder_Switch, SW3 Rotary_Encoder_Switch, U1 STM32F030F4Px, U2 RT9193, X2 SWD

Commit message: WIP
Parts:
- J1: footprint Connector_USB:USB_B_OST_USB-B1HSxx_Horizontal -> controller:USB_B_OST_USB-B1HSxx_Horizontal
- SW1, SW2, SW3: footprint Rotary_Encoder:RotaryEncoder_Alps_EC12E-Switch_Vertical_H20mm -> device.farm:RotaryEncoder_Bourns_PEC12R-4x20F-Sxxxx
