File: controller/controller.sch (KiCad schematic (older format))
At the start: 18 parts, among them J1 USB_B, J2 Conn_01x03, SW1 Rotary_Encoder_Switch, SW2 Rotary_Encoder_Switch, SW3 Rotary_Encoder_Switch, U1 STM32F030F4Px, U2 RT9193, X2 SWD

Commit message: WIP
Parts:
- J1: footprint Connector_USB:USB_B_OST_USB-B1HSxx_Horizontal -> controller:USB_B_OST_USB-B1HSxx_Horizontal
Changed lines of the file:
@@
 F 0 "J1" H 3155 4667 50  0000 C CNN
 F 1 "USB_B" H 3155 4576 50  0000 C CNN
-F 2 "Connector_USB:USB_B_OST_USB-B1HSxx_Horizontal" H 3250 4150 50  0001 C CNN
+F 2 "controller:USB_B_OST_USB-B1HSxx_Horizontal" H 3250 4150 50  0001 C CNN
 F 3 " ~" H 3250 4150 50  0001 C CNN
 	1    3100 4200
